Commit message: 🐛 fix(mecanum_sim): replace virtual link with body to adapt for fastlio.

File: moudles/mecanum_car/robot.urdf (robot description, URDF)
Before this commit: robot mecanum_robot, 13 links, 12 joints
Links:
- removed link base_footprint
- added link body
Joints:
- removed joint base_footprint_to_chassis
- added joint body_to_chassis: type fixed, parent body, child chassis, origin xyz=0 0 0.225 rpy=0 0 0
